Commit message: update scout

File: robot_simulation/urdf/mini.xacro (robot description, xacro)
@@ -4,8 +4,8 @@
     <xacro:arg name="robot_namespace" default="/" />
     <xacro:arg name="urdf_extras" default="empty.urdf" />
-    <xacro:include filename="$(find scout_description)/urdf/scout_mini_wheel_1.xacro" />
-    <xacro:include filename="$(find scout_description)/urdf/scout_mini_wheel_2.xacro" />
-    <xacro:include filename="$(find scout_description)/urdf/scout_mini_wheel_3.xacro" />
-    <xacro:include filename="$(find scout_description)/urdf/scout_mini_wheel_4.xacro" />
+    <xacro:include filename="$(find robot_simulation)/urdf/scout_mini_wheel_1.xacro" />
+    <xacro:include filename="$(find robot_simulation)/urdf/scout_mini_wheel_2.xacro" />
+    <xacro:include filename="$(find robot_simulation)/urdf/scout_mini_wheel_3.xacro" />
+    <xacro:include filename="$(find robot_simulation)/urdf/scout_mini_wheel_4.xacro" />
     <xacro:include filename="$(find robot_simulation)/urdf/VLP-16.urdf.xacro" />
     <!-- Variables -->
@@ -31,8 +31,8 @@
         <child link="base_footprint" />
     </joint> -->
-    <link name="dummy_baselink"/>
-    <joint name="dummy_baselink_joint" type="fixed">
+    <link name="dummy_base_link"/>
+    <joint name="dummy_base_link_joint" type="fixed">
         <origin xyz="0 0 0" rpy="0 0 0" />
-        <parent link="dummy_baselink" />
+        <parent link="dummy_base_link" />
         <child link="base_link" />
     </joint>
@@ -84,4 +84,10 @@
         <parent link="base_link" />
         <child link="box_link" />
+    </joint>
+    <link name="imu_link"/>
+    <joint name="imu_joint" type="fixed">
+        <origin xyz="0 0 0" rpy="0 0 0" />
+        <parent link="base_link" />
+        <child link="imu_link" />
     </joint>
     <!-- <link name="laser_link">
@@ -184,4 +190,4 @@
     <xacro:include filename="$(arg urdf_extras)" />
     <!-- Gazebo definitions  -->
-    <xacro:include filename="$(find scout_description)/urdf/scout_mini.gazebo" />
+    <xacro:include filename="$(find robot_simulation)/urdf/scout_mini.gazebo" />
 </robot>

Commit message: update path planning

File: robot_simulation/urdf/mini.xacro (robot description, xacro)
@@ -4,8 +4,8 @@
     <xacro:arg name="robot_namespace" default="/" />
     <xacro:arg name="urdf_extras" default="empty.urdf" />
-    <xacro:include filename="$(find robot_simulation)/urdf/scout_mini_wheel_1.xacro" />
-    <xacro:include filename="$(find robot_simulation)/urdf/scout_mini_wheel_2.xacro" />
-    <xacro:include filename="$(find robot_simulation)/urdf/scout_mini_wheel_3.xacro" />
-    <xacro:include filename="$(find robot_simulation)/urdf/scout_mini_wheel_4.xacro" />
+    <xacro:include filename="$(find scout_description)/urdf/scout_mini_wheel_1.xacro" />
+    <xacro:include filename="$(find scout_description)/urdf/scout_mini_wheel_2.xacro" />
+    <xacro:include filename="$(find scout_description)/urdf/scout_mini_wheel_3.xacro" />
+    <xacro:include filename="$(find scout_description)/urdf/scout_mini_wheel_4.xacro" />
     <xacro:include filename="$(find robot_simulation)/urdf/VLP-16.urdf.xacro" />
     <!-- Variables -->
@@ -33,5 +33,5 @@
     <link name="dummy_base_link"/>
     <joint name="dummy_base_link_joint" type="fixed">
-        <origin xyz="0 0 0" rpy="0 0 0" />
+        <origin xyz="0 0 0.18" rpy="0 0 0" />
         <parent link="dummy_base_link" />
         <child link="base_link" />
